Commit message: feat: port simulation to Gazebo Fortress (gz-sim) + headless demo video
Gazebo Classic ROS packages are EOL/removed from the Humble apt repo, so the
simulation layer is reimplemented on Ignition/Gazebo Fortress via ros_gz:

- URDF gz-sim plugins: DiffDrive, OdometryPublisher-free wheel odom, gpu_lidar,
  rgbd_camera, navsat (GPS); sensor frame_ids set to the URDF links.
- course.sdf world (was course.world) with gz-sim systems + GPS georeference.
- ros_gz_bridge config bridging /clock /cmd_vel /odom /tf /scan /gps/fix /camera/*.
- Multi-arch Dockerfile (ros:humble base) + headless recorder (docker/).
- Centered drive wheels + dual casters; pure-arcing reactive controller with
  latched obstacle avoidance; waypoint route through the obstacle field.
- Fix: wrap xacro robot_description in ParameterValue(str); rename description
  launch args to avoid gui/rviz config leakage from parent launch files.
- media/demo.mp4: headless RViz recording of the autonomous run (see README
  note on gz-sim wheel-slip / odometry-frame visualization).

File: src/robot_description/urdf/robot.gazebo.xacro (robot description, xacro)
@@ -1,92 +1,75 @@
 <?xml version="1.0"?>
 <!--
-  Gazebo-specific description: material colours, surface friction, and the
-  ROS 2 sensor/actuator plugins (all from gazebo_ros_pkgs, Humble):
-    * differential drive  -> publishes /odom (+ TF), subscribes /cmd_vel
-    * 2D lidar (ray)       -> publishes /scan
-    * RGB-D depth camera   -> publishes /camera/{image_raw,depth/*,points}
-    * GPS                  -> publishes /gps/fix (sensor_msgs/NavSatFix)
+  Gazebo-specific description for Ignition/Gazebo Fortress (gz-sim 6).
+  System plugins (diff drive, joint states) + sensors (gpu_lidar, rgbd_camera,
+  navsat). Sensor data is published on gz topics and bridged to ROS 2 by
+  ros_gz_bridge (see robot_gazebo/config/bridge.yaml):
+    * diff drive  -> /odom (+ /tf), subscribes /cmd_vel
+    * gpu_lidar   -> /scan
+    * rgbd_camera -> /camera/image, /camera/depth_image, /camera/points
+    * navsat      -> /gps/fix
 -->
 <robot xmlns:xacro="http://ros.org/wiki/xacro">
-  <!-- ============================ Materials (Gazebo) ============================ -->
-  <gazebo reference="base_link">
-    <material>Gazebo/Blue</material>
-  </gazebo>
+  <!-- ============================ Materials / friction ============================ -->
+  <gazebo reference="base_link"><material>Gazebo/Blue</material></gazebo>
   <gazebo reference="left_wheel_link">
     <material>Gazebo/Black</material>
-    <mu1>1.0</mu1>
-    <mu2>1.0</mu2>
-    <kp>1e6</kp>
+    <mu1>1.5</mu1>
+    <mu2>1.5</mu2>
+    <kp>1e5</kp>
     <kd>1.0</kd>
   </gazebo>
   <gazebo reference="right_wheel_link">
     <material>Gazebo/Black</material>
-    <mu1>1.0</mu1>
-    <mu2>1.0</mu2>
-    <kp>1e6</kp>
+    <mu1>1.5</mu1>
+    <mu2>1.5</mu2>
+    <kp>1e5</kp>
     <kd>1.0</kd>
   </gazebo>
-  <gazebo reference="caster_link">
-    <material>Gazebo/Grey</material>
-    <!-- Near-frictionless so the passive caster slides freely -->
+  <gazebo reference="front_caster_link">
+    <!-- Frictionless ball caster so the diff drive can turn freely -->
     <mu1>0.0</mu1>
     <mu2>0.0</mu2>
-    <kp>1e6</kp>
-    <kd>1.0</kd>
   </gazebo>
-  <gazebo reference="lidar_link">
-    <material>Gazebo/DarkGrey</material>
+  <gazebo reference="rear_caster_link">
+    <mu1>0.0</mu1>
+    <mu2>0.0</mu2>
   </gazebo>
-  <gazebo reference="camera_link">
-    <material>Gazebo/White</material>
-  </gazebo>
-  <gazebo reference="gps_link">
-    <material>Gazebo/Green</material>
-  </gazebo>
-  <!-- ============================ Differential drive ============================ -->
+  <!-- ============================ Diff drive + odometry + joint states ============================ -->
   <gazebo>
-    <plugin name="diff_drive" filename="libgazebo_ros_diff_drive.so">
-      <ros>
-        <namespace>/</namespace>
-      </ros>
-      <!-- wheels -->
-      <left_joint>left_wheel_joint</left_joint>
-      <right_joint>right_wheel_joint</right_joint>
-      <!-- kinematics (must match URDF) -->
+    <!-- Actuation: maps /cmd_vel to wheel velocities.
+         left/right joints are intentionally crossed: with the wheel axes as
+         defined, this makes a positive angular.z command rotate the robot
+         left (CCW) to match the odometry/controller convention. -->
+    <plugin filename="ignition-gazebo-diff-drive-system"
+            name="ignition::gazebo::systems::DiffDrive">
+      <left_joint>right_wheel_joint</left_joint>
+      <right_joint>left_wheel_joint</right_joint>
       <wheel_separation>0.34</wheel_separation>
-      <wheel_diameter>0.13</wheel_diameter>
-      <!-- limits -->
-      <max_wheel_torque>20.0</max_wheel_torque>
-      <max_wheel_acceleration>2.0</max_wheel_acceleration>
-      <!-- topics / frames -->
-      <command_topic>cmd_vel</command_topic>
-      <odometry_topic>odom</odometry_topic>
-      <odometry_frame>odom</odometry_frame>
-      <robot_base_frame>base_footprint</robot_base_frame>
-      <!-- output -->
-      <publish_odom>true</publish_odom>
-      <publish_odom_tf>true</publish_odom_tf>
-      <publish_wheel_tf>true</publish_wheel_tf>
-      <update_rate>50</update_rate>
+      <wheel_radius>0.065</wheel_radius>
+      <max_linear_acceleration>1.0</max_linear_acceleration>
+      <topic>cmd_vel</topic>
+      <odom_topic>odom</odom_topic>
+      <tf_topic>tf</tf_topic>
+      <frame_id>odom</frame_id>
+      <child_frame_id>base_footprint</child_frame_id>
+      <odom_publish_frequency>50</odom_publish_frequency>
     </plugin>
-  </gazebo>
-  <!-- ============================ Joint states ============================ -->
-  <gazebo>
-    <plugin name="joint_states" filename="libgazebo_ros_joint_state_publisher.so">
-      <ros>
-        <namespace>/</namespace>
-      </ros>
-      <update_rate>50</update_rate>
+    <plugin filename="ignition-gazebo-joint-state-publisher-system"
+            name="ignition::gazebo::systems::JointStatePublisher">
+      <topic>joint_states</topic>
       <joint_name>left_wheel_joint</joint_name>
       <joint_name>right_wheel_joint</joint_name>
     </plugin>
   </gazebo>
-  <!-- ============================ 2D Lidar ============================ -->
+  <!-- ============================ 2D Lidar (gpu_lidar) ============================ -->
   <gazebo reference="lidar_link">
-    <sensor name="lidar" type="ray">
-      <pose>0 0 0 0 0 0</pose>
-      <visualize>false</visualize>
+    <sensor name="lidar" type="gpu_lidar">
+      <topic>scan</topic>
+      <ignition_frame_id>lidar_link</ignition_frame_id>
       <update_rate>10</update_rate>
-      <ray>
+      <always_on>1</always_on>
+      <visualize>true</visualize>
+      <lidar>
         <scan>
           <horizontal>
@@ -96,4 +79,10 @@
             <max_angle>3.141592</max_angle>
           </horizontal>
+          <vertical>
+            <samples>1</samples>
+            <resolution>1.0</resolution>
+            <min_angle>0.0</min_angle>
+            <max_angle>0.0</max_angle>
+          </vertical>
         </scan>
         <range>
@@ -107,26 +96,19 @@
           <stddev>0.01</stddev>
         </noise>
-      </ray>
-      <plugin name="lidar_controller" filename="libgazebo_ros_ray_sensor.so">
-        <ros>
-          <namespace>/</namespace>
-          <remapping>~/out:=scan</remapping>
-        </ros>
-        <output_type>sensor_msgs/LaserScan</output_type>
-        <frame_name>lidar_link</frame_name>
-      </plugin>
+      </lidar>
     </sensor>
   </gazebo>
-  <!-- ============================ Depth camera ============================ -->
+  <!-- ============================ Depth camera (rgbd_camera) ============================ -->
   <gazebo reference="camera_link">
-    <sensor name="depth_camera" type="depth">
-      <pose>0 0 0 0 0 0</pose>
-      <visualize>false</visualize>
-      <update_rate>15</update_rate>
-      <camera name="astra">
-        <horizontal_fov>1.047198</horizontal_fov> <!-- ~60 deg -->
+    <sensor name="depth_camera" type="rgbd_camera">
+      <topic>camera</topic>
+      <ignition_frame_id>camera_optical_link</ignition_frame_id>
+      <update_rate>10</update_rate>
+      <always_on>1</always_on>
+      <camera>
+        <horizontal_fov>1.047198</horizontal_fov>
         <image>
-          <width>640</width>
-          <height>480</height>
+          <width>320</width>
+          <height>240</height>
           <format>R8G8B8</format>
         </image>
@@ -135,50 +117,14 @@
           <far>8.0</far>
         </clip>
-        <noise>
-          <type>gaussian</type>
-          <mean>0.0</mean>
-          <stddev>0.007</stddev>
-        </noise>
       </camera>
-      <plugin name="depth_camera_controller" filename="libgazebo_ros_camera.so">
-        <ros>
-          <namespace>/</namespace>
-        </ros>
-        <camera_name>camera</camera_name>
-        <frame_name>camera_optical_link</frame_name>
-        <hack_baseline>0.07</hack_baseline>
-        <min_depth>0.2</min_depth>
-        <max_depth>8.0</max_depth>
-      </plugin>
     </sensor>
   </gazebo>
-  <!-- ============================ GPS ============================ -->
+  <!-- ============================ GPS (navsat) ============================ -->
   <gazebo reference="gps_link">
-    <sensor name="gps" type="gps">
-      <always_on>true</always_on>
+    <sensor name="navsat" type="navsat">
+      <topic>gps/fix</topic>
+      <ignition_frame_id>gps_link</ignition_frame_id>
       <update_rate>5</update_rate>
-      <gps>
-        <position_sensing>
-          <horizontal>
-            <noise type="gaussian">
-              <mean>0.0</mean>
-              <stddev>0.8</stddev>   <!-- ~metre-level civilian GPS -->
-            </noise>
-          </horizontal>
-          <vertical>
-            <noise type="gaussian">
-              <mean>0.0</mean>
-              <stddev>1.5</stddev>
-            </noise>
-          </vertical>
-        </position_sensing>
-      </gps>
-      <plugin name="gps_controller" filename="libgazebo_ros_gps_sensor.so">
-        <ros>
-          <namespace>/</namespace>
-          <remapping>~/out:=gps/fix</remapping>
-        </ros>
-        <frame_name>gps_link</frame_name>
-      </plugin>
+      <always_on>1</always_on>
     </sensor>
   </gazebo>

File: src/robot_description/urdf/robot.urdf.xacro (robot description, xacro)
@@ -18,5 +18,5 @@
   <xacro:property name="wheel_mass"      value="0.5"/>
   <xacro:property name="wheel_separation" value="0.34"/>   <!-- centre-to-centre -->
-  <xacro:property name="wheel_xoff"      value="0.10"/>     <!-- forward of base centre -->
+  <xacro:property name="wheel_xoff"      value="0.0"/>      <!-- wheels centred under the CoM so the robot pivots cleanly in place -->
   <xacro:property name="wheel_zoff"      value="0.02"/>     <!-- drop below base centre -->
   <xacro:property name="caster_radius" value="0.045"/>
@@ -109,23 +109,29 @@
   <xacro:wheel prefix="left"  y_reflect="1"/>
   <xacro:wheel prefix="right" y_reflect="-1"/>
-  <!-- ============================ Caster ============================ -->
-  <link name="caster_link">
-    <visual>
-      <geometry><sphere radius="${caster_radius}"/></geometry>
-      <material name="caster_grey"><color rgba="0.4 0.4 0.4 1.0"/></material>
-    </visual>
-    <collision>
-      <geometry><sphere radius="${caster_radius}"/></geometry>
-    </collision>
-    <inertial>
-      <mass value="0.2"/>
-      <xacro:sphere_inertia m="0.2" r="${caster_radius}"/>
-    </inertial>
-  </link>
-  <joint name="caster_joint" type="fixed">
-    <parent link="base_link"/>
-    <child  link="caster_link"/>
-    <origin xyz="${-caster_xoff} 0 ${-(wheel_radius + wheel_zoff - caster_radius)}" rpy="0 0 0"/>
-  </joint>
+  <!-- ============================ Casters (front + rear) ============================ -->
+  <!-- With the drive wheels centred, two frictionless ball casters (front and
+       rear) keep the robot level fore-aft while letting it pivot in place. -->
+  <xacro:macro name="caster" params="prefix x_sign">
+    <link name="${prefix}_caster_link">
+      <visual>
+        <geometry><sphere radius="${caster_radius}"/></geometry>
+        <material name="caster_grey"><color rgba="0.4 0.4 0.4 1.0"/></material>
+      </visual>
+      <collision>
+        <geometry><sphere radius="${caster_radius}"/></geometry>
+      </collision>
+      <inertial>
+        <mass value="0.2"/>
+        <xacro:sphere_inertia m="0.2" r="${caster_radius}"/>
+      </inertial>
+    </link>
+    <joint name="${prefix}_caster_joint" type="fixed">
+      <parent link="base_link"/>
+      <child  link="${prefix}_caster_link"/>
+      <origin xyz="${x_sign * caster_xoff} 0 ${-(wheel_radius + wheel_zoff - caster_radius)}" rpy="0 0 0"/>
+    </joint>
+  </xacro:macro>
+  <xacro:caster prefix="front" x_sign="1"/>
+  <xacro:caster prefix="rear"  x_sign="-1"/>
   <!-- ============================ 2D Lidar ============================ -->
   <link name="lidar_link">
